File: hw/mini68k/mini68k.sch (KiCad schematic (older format))
At the start: 25 parts

Commit message: * oscillator, gal
Parts:
- added U?: GAL16V8, symbol GAL16V8
- added X?: TCXO-14, Oscillators:Oscillator_DIP-14, symbol TCXO-14
Connections:
- net A15: now also U?.3 (I3)
- net A16: now also U?.2 (I2)
- net GND: now also U?.10 (GND)
- net VCC: now also U?.20 (VCC)
- net AS: now reaches U?.28 (AS)
- net AS: now also U?.4 (I4)
- net DS: now reaches U?.29 (DS)
- net DS: now also U?.5 (I5)
Changed lines of the file:
@@
 LIBS:contrib
 LIBS:valves
+LIBS:Lattice
+LIBS:MAX708
+LIBS:Oscillators
 LIBS:mini68k-cache
 EELAYER 25 0
@@
 Wire Wire Line
 	9900 4700 9950 4700
+$Comp
+L GAL16V8 U?
+U 1 1 5B29ACED
+P 6050 2700
+F 0 "U?" H 5700 3350 50  0000 L CNN
+F 1 "GAL16V8" H 6100 3350 50  0000 L CNN
+F 2 "" H 6050 2700 50  0001 C CNN
+F 3 "" H 6050 2700 50  0001 C CNN
+	1    6050 2700
+	1    0    0    -1
+$EndComp
+Text GLabel 5500 2300 0    60   Input ~ 0
+A16
+Text GLabel 5500 2400 0    60   Input ~ 0
+A15
+Text GLabel 1250 3850 0    60   Output ~ 0
+AS
+Text GLabel 5500 2500 0    60   Input ~ 0
+AS
+Text GLabel 1250 3950 0    60   Output ~ 0
+DS
+Text GLabel 5500 2600 0    60   Input ~ 0
+DS
+Wire Wire Line
+	1250 3850 1300 3850
+Wire Wire Line
+	1250 3950 1300 3950
+Wire Wire Line
+	5500 2300 5550 2300
+Wire Wire Line
+	5500 2400 5550 2400
+Wire Wire Line
+	5500 2500 5550 2500
+Wire Wire Line
+	5500 2600 5550 2600
+$Comp
+L TCXO-14 X?
+U 1 1 5B29FF33
+P 4500 1350
+F 0 "X?" H 4300 1600 50  0000 L CNN
+F 1 "TCXO-14" H 4550 1100 50  0000 L CNN
+F 2 "Oscillators:Oscillator_DIP-14" H 4950 1000 50  0001 C CNN
+F 3 "" H 4400 1350 50  0001 C CNN
+	1    4500 1350
+	1    0    0    -1
+$EndComp
 $EndSCHEMATC

Commit message: everything but reset and i/o
Connections:
- net A1: now also U?.1 (RS1)
- net A2: now also U?.3 (RS2)
- net A3: now also U?.5 (RS3)
- net A4: now also U?.6 (RS4)
- net GND: now also U?.1 (GND), U?.11 (I10/~OE~), U?.20 (CS), U?.20 (~CS), X?.7 (GND)
- net INTR: now also U?.21 (IRQ)
- net VCC: now also U?.27 (WE), U?.8 (VCC), X?.14 (Vcc)
- net R/W: now reaches U?.30 (R/W)
- net R/W: now also U?.7 (I7), U?.8 (R/W)
- net DTACK: now reaches U?.31 (DTACK)
- net DTACK: now also RN?.5 (R4), U?.13 (IO7), U?.9 (DTACK)
- net CLK: now reaches U?.34 (CLK)
- net CLK: now also U?.32 (X1/CLK), X?.8 (OUT)
- net HALT: now reaches U?.36 (HALT)
- net HALT: now also U?.12 (IO8)
- net RESET: now reaches U?.37 (RESET)
- net RESET: now also RN?.6 (R5), U?.17 (I03), U?.34 (RESET)
- net FC2: now reaches U?.43 (FC2)
- net FC2: now also U?.9 (I9)
- net FC1: now reaches U?.44 (FC1)
- net FC1: now also U?.8 (I8)
- net FC0: now reaches U?.45 (FC0)
- net FC0: now also U?.6 (I6)
- net UART_CS: now reaches U?.35 (CS)
- net UART_CS: now also U?.19 (IO1)
- net IACK: now reaches U?.37 (IACK)
- net IACK: now also U?.18 (IO2)
- net RAM_OE: now reaches U?.22 (~OE)
- net RAM_OE: now also U?.16 (IO4)
- net RAM_WE: now reaches U?.27 (~WE)
- net RAM_WE: now also U?.15 (IO5)
- net ROM_OE: now reaches U?.22 (OE)
- net ROM_OE: now also U?.14 (IO6)
- no-connect marks 4 -> 23

Commit message: initial pcb layout
Parts:
- removed C? (x2): C, symbol C
- removed R?: R, symbol R
- removed U?: NE555, symbol NE555
- removed U? (x3): 74LS05, symbol 74LS05
- added C11: .1u, Capacitors_THT:C_Disc_D5.0mm_W2.5mm_P2.50mm, symbol C
- added D2: RED, LEDs:LED_D4.0mm, symbol LED
- added J2: FTDI header, Pin_Headers:Pin_Header_Straight_1x06_Pitch2.54mm, symbol Conn_01x06_Female
- added JP1: Jumper, Pin_Headers:Pin_Header_Straight_1x02_Pitch2.54mm, symbol Jumper
- added R1: 330R, Resistors_THT:R_Axial_DIN0207_L6.3mm_D2.5mm_P7.62mm_Horizontal, symbol R
- added U6: 74LS05, Housings_DIP:DIP-14_W7.62mm_LongPads, symbol 74LS05
- added U7: MAX708CPA+, Housings_DIP:DIP-8_W7.62mm_LongPads, symbol MAX708CPA+
- C1: renamed from C?; footprint (none) -> Capacitors_THT:CP_Radial_D5.0mm_P2.50mm
- C2: renamed from C?; footprint (none) -> Capacitors_THT:CP_Radial_D5.0mm_P2.00mm
- C3, C4, C5, C6, C7, C8: renamed from C?; footprint (none) -> Capacitors_THT:C_Disc_D5.0mm_W2.5mm_P2.50mm
- D1: renamed from D?; footprint (none) -> Diodes_THT:D_DO-35_SOD27_P10.16mm_Horizontal
- J1: renamed from J?; footprint (none) -> Connectors:BARREL_JACK
- SW1: renamed from SW?; footprint (none) -> Buttons_Switches_THT:SW_CuK_JS202011CQN_DPDT_Straight
- SW2: renamed from SW?; footprint (none) -> Buttons_Switches_THT:SW_TH_Tactile_Omron_B3F-10xx
- U1: renamed from U?; footprint DIP28 -> Housings_DIP:DIP-28_W15.24mm_LongPads
- U2: renamed from U?; footprint (none) -> Housings_DIP:DIP-48_W15.24mm_LongPads
- U3: renamed from U?; footprint (none) -> TO_SOT_Packages_THT:TO-220-3_Horizontal
- U4: renamed from U?; footprint (none) -> Housings_DIP:DIP-28_W15.24mm_LongPads
- U5: renamed from U?; footprint (none) -> Housings_DIP:DIP-20_W7.62mm_LongPads
- U8: renamed from U?; footprint (none) -> Housings_DIP:DIP-40_W15.24mm_LongPads
- gave numbers to parts that had none: 2
Connections:
- net DTACK: now also RN1.3 (R2); no longer RN1.5 (R4)
- net GND: now also C11.2, J2.1 (Pin_1), R1.1, U6.7 (GND), U6.7 (GND), U6.7 (GND), U6.7 (GND), U6.7 (GND), U6.7 (GND), U7.3 (GND), U7.4 (PFI)
- net INTR: now also RN1.5 (R4); no longer RN1.7 (R6)
- net RESET: now also RN1.4 (R3); no longer RN1.6 (R5)
- net TR: now also RN1.2 (R1); no longer RN1.4 (R3), SW2.1
- net VCC: now also C11.1, D2.2 (A), JP1.2, U6.14 (VCC), U6.14 (VCC), U6.14 (VCC), U6.14 (VCC), U6.14 (VCC), U6.14 (VCC), U7.2 (VCC)
- net TX1: now reaches U8.30 (TXDA)
- net TX1: now also J2.4 (Pin_4)
- net RX1: now reaches U8.31 (RXDA)
- net RX1: now also J2.5 (Pin_5)
- net RST: now reaches U5.1 (I1/CLK)
- net RST: now also U6.2
- new net: J2.3 (Pin_3), JP1.1
- new net: U6.1, U7.8 (RESET)
- new net: D2.1 (K), R1.2
- new net MR: SW2.1, U7.1 (*MR)
- no-connect marks 23 -> 35
Other:
- moved on the sheet: RN1, SW2

Commit message: initial layout
Connections:
- no-connect marks 35 -> 39
Changed lines of the file:
@@
 NoConn ~ 10300 6150
 NoConn ~ 10300 6500
+NoConn ~ 6900 6150
+NoConn ~ 6900 5750
+NoConn ~ 8450 6150
+NoConn ~ 8450 6250
 $EndSCHEMATC

Commit message: v2 fixes:
  - swapped rx/tx
  - reset switch
  - pullup RST
  - pin one of X1
  - remove VCC plane from under 7805
Parts:
- SW2: footprint Buttons_Switches_THT:SW_TH_Tactile_Omron_B3F-10xx -> Buttons_Switches_THT:SW_PUSH_6mm
Connections:
- net TR is gone; now on net RST: RN1.2 (R1)
- net RX1: now also J2.4 (Pin_4); no longer J2.5 (Pin_5)
- net TX1: now also J2.5 (Pin_5); no longer J2.4 (Pin_4)
Changed lines of the file:
@@
 Connection ~ 4900 4950
 $Comp
-L GND #PWR12
+L GND #PWR01
 U 1 1 5B285D6B
 P 3400 5450
-F 0 "#PWR12" H 3400 5200 50  0001 C CNN
+F 0 "#PWR01" H 3400 5200 50  0001 C CNN
 F 1 "GND" H 3400 5300 50  0000 C CNN
 F 2 "" H 3400 5450 50  0001 C CNN
@@
 $EndComp
 $Comp
-L GND #PWR10
+L GND #PWR02
 U 1 1 5B285D9E
 P 2950 5400
-F 0 "#PWR10" H 2950 5150 50  0001 C CNN
+F 0 "#PWR02" H 2950 5150 50  0001 C CNN
 F 1 "GND" H 2950 5250 50  0000 C CNN
 F 2 "" H 2950 5400 50  0001 C CNN
@@
 $EndComp
 $Comp
-L GND #PWR9
+L GND #PWR03
 U 1 1 5B285DCA
 P 2400 5400
-F 0 "#PWR9" H 2400 5150 50  0001 C CNN
+F 0 "#PWR03" H 2400 5150 50  0001 C CNN
 F 1 "GND" H 2400 5250 50  0000 C CNN
 F 2 "" H 2400 5400 50  0001 C CNN
@@
 $EndComp
 $Comp
-L VCC #PWR31
+L VCC #PWR04
 U 1 1 5B285DF8
 P 9000 5650
-F 0 "#PWR31" H 9000 5500 50  0001 C CNN
+F 0 "#PWR04" H 9000 5500 50  0001 C CNN
 F 1 "VCC" H 9000 5800 50  0000 C CNN
 F 2 "" H 9000 5650 50  0001 C CNN
@@
 $EndComp
 $Comp
-L VCC #PWR11
+L VCC #PWR05
 U 1 1 5B285E22
 P 3400 4750
-F 0 "#PWR11" H 3400 4600 50  0001 C CNN
+F 0 "#PWR05" H 3400 4600 50  0001 C CNN
 F 1 "VCC" H 3400 4900 50  0000 C CNN
 F 2 "" H 3400 4750 50  0001 C CNN
@@
 $EndComp
 $Comp
-L VCC #PWR6
+L VCC #PWR06
 U 1 1 5B285E55
 P 2200 800
-F 0 "#PWR6" H 2200 650 50  0001 C CNN
+F 0 "#PWR06" H 2200 650 50  0001 C CNN
 F 1 "VCC" H 2200 950 50  0000 C CNN
 F 2 "" H 2200 800 50  0001 C CNN
@@
 $EndComp
 $Comp
-L GND #PWR8
+L GND #PWR07
 U 1 1 5B285EAD
 P 2250 4300
-F 0 "#PWR8" H 2250 4050 50  0001 C CNN
+F 0 "#PWR07" H 2250 4050 50  0001 C CNN
 F 1 "GND" H 2250 4150 50  0000 C CNN
 F 2 "" H 2250 4300 50  0001 C CNN
@@
 	3400 4750 3400 4950
 $Comp
-L GND #PWR5
+L GND #PWR08
 U 1 1 5B285E81
 P 2150 4300
-F 0 "#PWR5" H 2150 4050 50  0001 C CNN
+F 0 "#PWR08" H 2150 4050 50  0001 C CNN
 F 1 "GND" H 2150 4150 50  0000 C CNN
 F 2 "" H 2150 4300 50  0001 C CNN
@@
 	1250 5050 1300 5050
 $Comp
-L GND #PWR2
+L GND #PWR09
 U 1 1 5B28799F
 P 1400 5400
-F 0 "#PWR2" H 1400 5150 50  0001 C CNN
+F 0 "#PWR09" H 1400 5150 50  0001 C CNN
 F 1 "GND" H 1400 5250 50  0000 C CNN
 F 2 "" H 1400 5400 50  0001 C CNN
@@
 Connection ~ 1400 5250
 $Comp
-L VCC #PWR1
+L VCC #PWR010
 U 1 1 5B287FD8
 P 750 900
-F 0 "#PWR1" H 750 750 50  0001 C CNN
+F 0 "#PWR010" H 750 750 50  0001 C CNN
 F 1 "VCC" H 750 1050 50  0000 C CNN
 F 2 "" H 750 900 50  0001 C CNN
@@
 F 0 "SW2" H 7500 5100 50  0000 L CNN
 F 1 "SW_Push" H 7450 4940 50  0000 C CNN
-F 2 "Buttons_Switches_THT:SW_TH_Tactile_Omron_B3F-10xx" H 7450 5200 50  0001 C CNN
+F 2 "Buttons_Switches_THT:SW_PUSH_6mm" H 7450 5200 50  0001 C CNN
 F 3 "" H 7450 5200 50  0001 C CNN
 	1    7450 5000
@@
 $EndComp
 $Comp
-L GND #PWR28
+L GND #PWR011
 U 1 1 5B28B46E
 P 7750 5000
-F 0 "#PWR28" H 7750 4750 50  0001 C CNN
+F 0 "#PWR011" H 7750 4750 50  0001 C CNN
 F 1 "GND" H 7750 4850 50  0000 C CNN
 F 2 "" H 7750 5000 50  0001 C CNN
@@
 Wire Wire Line
 	7750 5000 7650 5000
-Text GLabel 8400 5750 0    60   Input ~ 0
-TR
 Wire Wire Line
 	8400 5950 8450 5950
@@
 	5500 3000 5550 3000
 $Comp
-L GND #PWR21
+L GND #PWR012
 U 1 1 5B2A926F
 P 5500 3150
-F 0 "#PWR21" H 5500 2900 50  0001 C CNN
+F 0 "#PWR012" H 5500 2900 50  0001 C CNN
 F 1 "GND" H 5500 3000 50  0000 C CNN
 F 2 "" H 5500 3150 50  0001 C CNN
@@
 	4800 1350 4850 1350
 $Comp
-L GND #PWR17
+L GND #PWR013
 U 1 1 5B2A991F
 P 4500 1700
-F 0 "#PWR17" H 4500 1450 50  0001 C CNN
+F 0 "#PWR013" H 4500 1450 50  0001 C CNN
 F 1 "GND" H 4500 1550 50  0000 C CNN
 F 2 "" H 4500 1700 50  0001 C CNN
@@
 	4500 1650 4500 1700
 $Comp
-L VCC #PWR16
+L VCC #PWR014
 U 1 1 5B2A9A2D
 P 4500 950
-F 0 "#PWR16" H 4500 800 50  0001 C CNN
+F 0 "#PWR014" H 4500 800 50  0001 C CNN
 F 1 "VCC" H 4500 1100 50  0000 C CNN
 F 2 "" H 4500 950 50  0001 C CNN
@@
 $EndComp
 $Comp
-L VCC #PWR29
+L VCC #PWR015
 U 1 1 5B2A9A89
 P 9000 900
-F 0 "#PWR29" H 9000 750 50  0001 C CNN
+F 0 "#PWR015" H 9000 750 50  0001 C CNN
 F 1 "VCC" H 9000 1050 50  0000 C CNN
 F 2 "" H 9000 900 50  0001 C CNN
@@
 $EndComp
 $Comp
-L VCC #PWR23
+L VCC #PWR016
 U 1 1 5B2A9AE5
 P 6050 2050
-F 0 "#PWR23" H 6050 1900 50  0001 C CNN
+F 0 "#PWR016" H 6050 1900 50  0001 C CNN
 F 1 "VCC" H 6050 2200 50  0000 C CNN
 F 2 "" H 6050 2050 50  0001 C CNN
@@
 	6050 2100 6050 2050
 $Comp
-L GND #PWR24
+L GND #PWR017
 U 1 1 5B2A9BF4
 P 6050 3350
-F 0 "#PWR24" H 6050 3100 50  0001 C CNN
+F 0 "#PWR017" H 6050 3100 50  0001 C CNN
 F 1 "GND" H 6050 3200 50  0000 C CNN
 F 2 "" H 6050 3350 50  0001 C CNN
@@
 $EndComp
 $Comp
-L GND #PWR30
+L GND #PWR018
 U 1 1 5B2A9C8C
 P 9000 3600
-F 0 "#PWR30" H 9000 3350 50  0001 C CNN
+F 0 "#PWR018" H 9000 3350 50  0001 C CNN
 F 1 "GND" H 9000 3450 50  0000 C CNN
 F 2 "" H 9000 3600 50  0001 C CNN
@@
 	9000 3600 9000 3550
 $Comp
-L VCC #PWR19
+L VCC #PWR019
 U 1 1 5B2AA14D
 P 4700 5600
-F 0 "#PWR19" H 4700 5450 50  0001 C CNN
+F 0 "#PWR019" H 4700 5450 50  0001 C CNN
 F 1 "VCC" H 4700 5750 50  0000 C CNN
 F 2 "" H 4700 5600 50  0001 C CNN
@@
 $EndComp
 $Comp
-L VCC #PWR3
+L VCC #PWR020
 U 1 1 5B2AA1A9
 P 1650 5750
-F 0 "#PWR3" H 1650 5600 50  0001 C CNN
+F 0 "#PWR020" H 1650 5600 50  0001 C CNN
 F 1 "VCC" H 1650 5900 50  0000 C CNN
 F 2 "" H 1650 5750 50  0001 C CNN
@@
 $EndComp
 $Comp
-L GND #PWR20
+L GND #PWR021
 U 1 1 5B2AA205
 P 4700 7700
-F 0 "#PWR20" H 4700 7450 50  0001 C CNN
+F 0 "#PWR021" H 4700 7450 50  0001 C CNN
 F 1 "GND" H 4700 7550 50  0000 C CNN
 F 2 "" H 4700 7700 50  0001 C CNN
@@
 $EndComp
 $Comp
-L GND #PWR4
+L GND #PWR022
 U 1 1 5B2AA261
 P 1650 7550
-F 0 "#PWR4" H 1650 7300 50  0001 C CNN
+F 0 "#PWR022" H 1650 7300 50  0001 C CNN
 F 1 "GND" H 1650 7400 50  0000 C CNN
 F 2 "" H 1650 7550 50  0001 C CNN
@@
 	2250 6900 2150 6900
 $Comp
-L GND #PWR7
+L GND #PWR023
 U 1 1 5B2ACC50
 P 2200 7100
-F 0 "#PWR7" H 2200 6850 50  0001 C CNN
+F 0 "#PWR023" H 2200 6850 50  0001 C CNN
 F 1 "GND" H 2200 6950 50  0000 C CNN
 F 2 "" H 2200 7100 50  0001 C CNN
@@
 	3950 7450 4000 7450
 $Comp
-L GND #PWR15
+L GND #PWR024
 U 1 1 5B2AD0B0
 P 3950 7600
-F 0 "#PWR15" H 3950 7350 50  0001 C CNN
+F 0 "#PWR024" H 3950 7350 50  0001 C CNN
 F 1 "GND" H 3950 7450 50  0000 C CNN
 F 2 "" H 3950 7600 50  0001 C CNN
@@
 	3950 7550 3950 7600
 $Comp
-L VCC #PWR14
+L VCC #PWR025
 U 1 1 5B2AD1E7
 P 3900 7350
-F 0 "#PWR14" H 3900 7200 50  0001 C CNN
+F 0 "#PWR025" H 3900 7200 50  0001 C CNN
 F 1 "VCC" H 3900 7500 50  0000 C CNN
 F 2 "" H 3900 7350 50  0001 C CNN
@@
 	6050 3350 6050 3300
 $Comp
-L GND #PWR26
+L GND #PWR026
 U 1 1 5B2B5101
 P 6950 6300
-F 0 "#PWR26" H 6950 6050 50  0001 C CNN
+F 0 "#PWR026" H 6950 6050 50  0001 C CNN
 F 1 "GND" H 6950 6150 50  0000 C CNN
 F 2 "" H 6950 6300 50  0001 C CNN
@@
 $EndComp
 Connection ~ 5200 4950
-Text GLabel 6950 5950 2    60   Input ~ 0
+Text GLabel 6950 5850 2    60   Input ~ 0
 TX1
 $Comp
@@
 Wire Wire Line
 	6900 5950 6950 5950
-Text GLabel 6950 5850 2    60   Input ~ 0
+Text GLabel 6950 5950 2    60   Input ~ 0
 RX1
 Wire Wire Line
@@
 	6900 6050 6950 6050
 $Comp
-L VCC #PWR27
+L VCC #PWR027
 U 1 1 5B2B71ED
 P 7600 6050
-F 0 "#PWR27" H 7600 5900 50  0001 C CNN
+F 0 "#PWR027" H 7600 5900 50  0001 C CNN
 F 1 "VCC" H 7600 6200 50  0000 C CNN
 F 2 "" H 7600 6050 50  0001 C CNN
@@
 	7250 5000 7150 5000
 $Comp
-L GND #PWR25
+L GND #PWR028
 U 1 1 5B2D247C
 P 6100 4550
-F 0 "#PWR25" H 6100 4300 50  0001 C CNN
+F 0 "#PWR028" H 6100 4300 50  0001 C CNN
 F 1 "GND" H 6100 4400 50  0000 C CNN
 F 2 "" H 6100 4550 50  0001 C CNN
@@
 Connection ~ 6100 4500
 $Comp
-L VCC #PWR22
+L VCC #PWR029
 U 1 1 5B2D268D
 P 5900 4050
-F 0 "#PWR22" H 5900 3900 50  0001 C CNN
+F 0 "#PWR029" H 5900 3900 50  0001 C CNN
 F 1 "VCC" H 5900 4200 50  0000 C CNN
 F 2 "" H 5900 4050 50  0001 C CNN
@@
 $EndComp
 $Comp
-L GND #PWR18
+L GND #PWR030
 U 1 1 5B2D3BF8
 P 4700 3100
-F 0 "#PWR18" H 4700 2850 50  0001 C CNN
+F 0 "#PWR030" H 4700 2850 50  0001 C CNN
 F 1 "GND" H 4700 2950 50  0000 C CNN
 F 2 "" H 4700 3100 50  0001 C CNN
@@
 	4200 3050 4300 3050
 $Comp
-L VCC #PWR13
+L VCC #PWR031
 U 1 1 5B2D3EF5
 P 3800 3050
-F 0 "#PWR13" H 3800 2900 50  0001 C CNN
+F 0 "#PWR031" H 3800 2900 50  0001 C CNN
 F 1 "VCC" H 3800 3200 50  0000 C CNN
 F 2 "" H 3800 3050 50  0001 C CNN
@@
 NoConn ~ 8450 6150
 NoConn ~ 8450 6250
+Text GLabel 8400 5750 0    60   Input ~ 0
+RST
 $EndSCHEMATC

Commit message: KiCad 5
Parts:
- C1, C2: symbol CP1 -> Device:CP1
- C11, C3, C4, C5, C6, C7, C8: symbol C -> Device:C
- D1: symbol D_ALT -> Device:D_ALT
- D2: symbol LED -> Device:LED
- J1: symbol Jack-DC -> mini68k-rescue:Jack-DC
- J2: symbol Conn_01x06_Female -> mini68k-rescue:Conn_01x06_Female
- JP1: symbol Jumper -> Device:Jumper
- R1: symbol R -> Device:R
- RN1: symbol R_Network06 -> Device:R_Network06
- SW1: symbol SW_SPDT -> mini68k-rescue:SW_SPDT
- SW2: symbol SW_Push -> mini68k-rescue:SW_Push
- U1: symbol HM62256BLP-7 -> mini68k-rescue:HM62256BLP-7
- U2: symbol 68008D -> mini68k-rescue:68008D
- U3: symbol L7805 -> mini68k-rescue:L7805
- U4: symbol 28C256 -> mini68k-rescue:28C256
- U5: symbol GAL16V8 -> mini68k-rescue:GAL16V8
- U6: symbol 74LS05 -> mini68k-rescue:74LS05
- U7: symbol MAX708CPA+ -> mini68k-rescue:MAX708CPA+
- U8: symbol 68681 -> mini68k-rescue:68681
- X1: symbol TCXO-14 -> mini68k-rescue:TCXO-14
Connections:
- net RX2: now reaches U8.10 (RXDB)
- net TX2: now reaches U8.11 (TXDB)
- net OP1: now reaches U8.12 (OP1)
- net OP3: now reaches U8.13 (OP3)
- net OP5: now reaches U8.14 (OP5)
- net OP7: now reaches U8.15 (OP7)
- net IP3: now reaches U8.2 (IP3)
- net OP6: now reaches U8.26 (OP6)
- net OP4: now reaches U8.27 (OP4)
- net OP2: now reaches U8.28 (OP2)
- net OP0: now reaches U8.29 (OP0)
- net IP2: now reaches U8.36 (IP2)
- net IP5: now reaches U8.38 (IP5)
- net IP4: now reaches U8.39 (IP4)
- net IP1: now reaches U8.4 (IP1)
- net IP0: now reaches U8.7 (IP0)
- no-connect marks 39 -> 23
Other:
- moved on the sheet: R1, SW2, U5, U6A, U7
